Commit message: [Model]: new model and example

File: mujoco_ros2_control_demos/urdf/test_diff_drive.xacro.urdf (robot description, URDF)
Before this commit: robot diff_drive, 4 links, 3 joints
Links:
- added link world
Joints:
- added joint world_to_base: type fixed, parent world, child chassis, origin xyz=0 0 1 rpy=0 0 0
